Commit message: Updated files

File: mycobot_ros2/mycobot_description/urdf/mycobot_280_m5/mycobot_280_m5_with_camera_flange.urdf (robot description, URDF)
Before this commit: robot firefighter, 9 links, 8 joints
Joints:
- joint joint6output_to_camera_flange: origin xyz=0 0 0.01 rpy=1.579 0 0 -> xyz=0 0 0.01 rpy=0 0 0
